File: Electronics/MidiControllerV2/SSD1306Oled.sch (KiCad schematic (older format))
At the start: 0 parts

Commit message: #32 Laid out rev1 schematic
Parts:
- added J?: Conn_01x04_Male, symbol Connector:Conn_01x04_Male
Connections:
- net +3.3V: now also J?.2 (Pin_2)
- net GND: now also J?.1 (Pin_1)
- net SCL: now also J?.3 (Pin_3)
- net SDA: now also J?.4 (Pin_4)
Changed lines of the file:
@@
 Comment4 ""
 $EndDescr
-Text HLabel 4100 3150 0    50   Input ~ 0
+Text HLabel 4400 3150 2    50   Input ~ 0
 GND
-Text HLabel 4050 3300 0    50   Input ~ 0
+Text HLabel 4400 3250 2    50   Input ~ 0
 +3.3V
-Text HLabel 3900 3650 0    50   Input ~ 0
+Text HLabel 4400 3450 2    50   Input ~ 0
 SDA
-Text HLabel 3850 3900 0    50   Input ~ 0
+Text HLabel 4400 3350 2    50   Input ~ 0
 SCL
+$Comp
+L Connector:Conn_01x04_Male J?
+U 1 1 5FFD7370
+P 4200 3250
+AR Path="/5FD44F32/5FFD7370" Ref="J?"  Part="1"
+AR Path="/60074587/5FFD7370" Ref="J?"  Part="1"
+F 0 "J?" H 4308 3531 50  0000 C CNN
+F 1 "Conn_01x04_Male" H 4308 3440 50  0000 C CNN
+F 2 "" H 4200 3250 50  0001 C CNN
+F 3 "~" H 4200 3250 50  0001 C CNN
+	1    4200 3250
+	1    0    0    -1
+$EndComp
 $EndSCHEMATC
