File: Electronics/MidiControllerV2/MidiControllerV2.sch (KiCad schematic (older format))
At the start: 22 parts

Commit message: #32 Laid out rev1 schematic
Parts:
- removed C?: C, symbol Device:C
- removed D?: LED, symbol Device:LED
- removed R? (x8): R, symbol Device:R
- removed SW?: Rotary_Encoder_Switch, symbol Device:Rotary_Encoder_Switch
- added C? (x10): C, symbol Device:C
- added D?: LED, symbol Device:LED
- added J?: BOOT1_H, symbol Connector:Conn_01x03_Male
- added J?: BOOT0_H, symbol Connector:Conn_01x03_Male
- added R? (x12): R, symbol Device:R
- added SW?: Encoder, symbol Device:Rotary_Encoder_Switch
- added SW?: SW_DPST, symbol Switch:SW_DPST
- SW?: value Rotary_Encoder_Switch -> Encoder
Connections:
- net +3V3: now reaches U?.1 (VBAT)
- net +3V3: now also J?.1 (Pin_1), R?.1, R?.2, U?.2 (VO), U?.24 (VDD), U?.36 (VDD), U?.48 (VDD), U?.9 (VDDA), C?.1, C?.1, C?.1, C?.1, C?.1, C?.1, J?.1 (Pin_1), J?.3 (Pin_3), R?.1, R?.2, R?.2, R?.2, R?.2, R?.2
- net ENC1B: now reaches U?.10 (PA0)
- net ENC1B: now also SW?.B, R?.1
- net ENC1A: now reaches U?.11 (PA1)
- net ENC1A: now also SW?.A, R?.1
- net KP_R1: now reaches U?.12 (PA2)
- net KP_R2: now reaches U?.13 (PA3)
- net KP_R3: now reaches U?.14 (PA4)
- net KP_R4: now reaches U?.15 (PA5)
- net ENC2B: now reaches U?.16 (PA6)
- net ENC2B: now also R?.1, SW?.B
- net ENC2A: now reaches U?.17 (PA7)
- net ENC2A: now also R?.1, SW?.A
- net ENC2_SW: now reaches U?.19 (PB1)
- net ENC2_SW: now also C?.1, R?.1, SW?.S1
- net BOOT1: now reaches U?.20 (PB2)
- net BOOT1: now also R?.1
- net GND: now reaches U?.23 (VSS)
- net GND: now also C?.2, C?.2, C?.2, J?.2 (Pin_2), J?.4 (ID), J?.5 (GND), J?.6 (Shield), SW?.C, SW?.S2, U?.1 (GND), U?.35 (VSS), U?.47 (VSS), U?.8 (VSSA), C?.2, C?.2, C?.2, C?.2, C?.2, C?.2, C?.2, C?.2, C?.2, C?.2, D?.1 (K), J?.1 (Pin_1), J?.3 (Pin_3), SW?.1, SW?.3, SW?.C, SW?.S2
- net KP_C1: now reaches U?.25 (PB12)
- net KP_C2: now reaches U?.26 (PB13)
- net KP_C3: now reaches U?.27 (PB14)
- net KP_C4: now reaches U?.28 (PB15)
- net ENC1_SW: now reaches U?.3 (PC14)
- net ENC1_SW: now also C?.1, R?.1, SW?.S1
- net USBD-: now reaches U?.32 (PA11)
- net USBD-: now also R?.1
- net USBD+: now reaches U?.33 (PA12)
- net USBD+: now also R?.1, R?.2
- net SWDIO: now reaches U?.34 (PA13)
- net SWDIO: now also J?.3 (Pin_3)
- net SWDCLK: now reaches U?.37 (PA14)
- net SWDCLK: now also J?.4 (Pin_4)
- net OLED_SCL: now reaches U?.42 (PB6)
- net OLED_SDA: now reaches U?.43 (PB7)
- net BOOT0: now reaches U?.44 (BOOT0)
- net BOOT0: now also R?.2
- net OSCIN: now reaches U?.5 (PD0)
- net OSCIN: now also C?.1, Y?.1, R?.2
- net OSCOUT: now reaches U?.6 (PD1)
- net OSCOUT: now also C?.1, Y?.2, R?.1
- net RESET: now reaches U?.7 (NRST)
- net RESET: now also C?.1, R?.2, SW?.2, SW?.4
- net +5V: now reaches J?.1 (VBUS)
- net +5V: now also U?.3 (VI), C?.1, C?.1, R?.1
- net at J?.2 (D-): now also R?.2
- net at J?.3 (D+): now also R?.2
- net at R?.2: now also D?.2 (A)
- new net: J?.2 (Pin_2), R?.2
- new net: J?.2 (Pin_2), R?.1
Other:
- moved on the sheet: C?, J?, R?, SW?, U?, Y?

Commit message: #32 Pcb v2 components placed
Parts:
- C? (x10), R?: footprint (none) -> Capacitor_SMD:C_1206_3216Metric
- D?: footprint (none) -> LED_SMD:LED_1206_3216Metric
- R? (x13): footprint (none) -> Resistor_SMD:R_1206_3216Metric
- SW? (x2): footprint (none) -> Rotary_Encoder:RotaryEncoder_Alps_EC11E-Switch_Vertical_H20mm
- Y?: footprint (none) -> Crystal:Crystal_HC18-U_Vertical
Changed lines of the file:
@@
 F 0 "Y?" H 3500 1968 50  0000 C CNN
 F 1 "Crystal" H 3500 1877 50  0000 C CNN
-F 2 "" H 3500 1700 50  0001 C CNN
+F 2 "Crystal:Crystal_HC18-U_Vertical" H 3500 1700 50  0001 C CNN
 F 3 "~" H 3500 1700 50  0001 C CNN
 	1    3500 1700
@@
 F 0 "C?" H 3315 2246 50  0000 L CNN
 F 1 "C" H 3315 2155 50  0000 L CNN
-F 2 "" H 3238 2050 50  0001 C CNN
+F 2 "Capacitor_SMD:C_1206_3216Metric" H 3238 2050 50  0001 C CNN
 F 3 "~" H 3200 2200 50  0001 C CNN
 	1    3200 2200
@@
 F 0 "C?" H 3865 2246 50  0000 L CNN
 F 1 "C" H 3865 2155 50  0000 L CNN
-F 2 "" H 3788 2050 50  0001 C CNN
+F 2 "Capacitor_SMD:C_1206_3216Metric" H 3788 2050 50  0001 C CNN
 F 3 "~" H 3750 2200 50  0001 C CNN
 	1    3750 2200
@@
 F 0 "R?" H 9970 3296 50  0000 L CNN
 F 1 "R" H 9970 3205 50  0000 L CNN
-F 2 "" V 9830 3250 50  0001 C CNN
+F 2 "Resistor_SMD:R_1206_3216Metric" V 9830 3250 50  0001 C CNN
 F 3 "~" H 9900 3250 50  0001 C CNN
 	1    9900 3250
@@
 F 0 "R?" H 8270 1496 50  0000 L CNN
 F 1 "R" H 8270 1405 50  0000 L CNN
-F 2 "" V 8130 1450 50  0001 C CNN
+F 2 "Resistor_SMD:R_1206_3216Metric" V 8130 1450 50  0001 C CNN
 F 3 "~" H 8200 1450 50  0001 C CNN
 	1    8200 1450
@@
 F 0 "SW?" H 9100 3900 50  0000 L CNN
 F 1 "Encoder" H 9100 3800 50  0000 L CNN
-F 2 "" H 9150 3660 50  0001 C CNN
+F 2 "Rotary_Encoder:RotaryEncoder_Alps_EC11E-Switch_Vertical_H20mm" H 9150 3660 50  0001 C CNN
 F 3 "~" H 9300 3760 50  0001 C CNN
 	1    9300 3500
@@
 F 0 "R?" V 8550 3350 50  0000 C CNN
 F 1 "R" V 8650 3350 50  0000 C CNN
-F 2 "" V 8580 3350 50  0001 C CNN
+F 2 "Resistor_SMD:R_1206_3216Metric" V 8580 3350 50  0001 C CNN
 F 3 "~" H 8650 3350 50  0001 C CNN
 	1    8650 3350
@@
 F 0 "R?" V 8443 3650 50  0000 C CNN
 F 1 "R" V 8650 3650 50  0000 C CNN
-F 2 "" V 8580 3650 50  0001 C CNN
+F 2 "Resistor_SMD:R_1206_3216Metric" V 8580 3650 50  0001 C CNN
 F 3 "~" H 8650 3650 50  0001 C CNN
 	1    8650 3650
@@
 F 0 "R?" H 9970 5046 50  0000 L CNN
 F 1 "R" H 9970 4955 50  0000 L CNN
-F 2 "" V 9830 5000 50  0001 C CNN
+F 2 "Resistor_SMD:R_1206_3216Metric" V 9830 5000 50  0001 C CNN
 F 3 "~" H 9900 5000 50  0001 C CNN
 	1    9900 5000
@@
 F 0 "SW?" H 9100 5650 50  0000 L CNN
 F 1 "Encoder" H 9100 5550 50  0000 L CNN
-F 2 "" H 9150 5410 50  0001 C CNN
+F 2 "Rotary_Encoder:RotaryEncoder_Alps_EC11E-Switch_Vertical_H20mm" H 9150 5410 50  0001 C CNN
 F 3 "~" H 9300 5510 50  0001 C CNN
 	1    9300 5250
@@
 F 0 "R?" V 8443 5100 50  0000 C CNN
 F 1 "R" V 8534 5100 50  0000 C CNN
-F 2 "" V 8580 5100 50  0001 C CNN
+F 2 "Resistor_SMD:R_1206_3216Metric" V 8580 5100 50  0001 C CNN
 F 3 "~" H 8650 5100 50  0001 C CNN
 	1    8650 5100
@@
 F 0 "R?" V 8443 5400 50  0000 C CNN
 F 1 "R" V 8534 5400 50  0000 C CNN
-F 2 "" V 8580 5400 50  0001 C CNN
+F 2 "Resistor_SMD:R_1206_3216Metric" V 8580 5400 50  0001 C CNN
 F 3 "~" H 8650 5400 50  0001 C CNN
 	1    8650 5400
@@
 F 0 "R?" V 1950 1950 50  0000 C CNN
 F 1 "R" V 1850 1950 50  0000 C CNN
-F 2 "" V 1780 1950 50  0001 C CNN
+F 2 "Resistor_SMD:R_1206_3216Metric" V 1780 1950 50  0001 C CNN
 F 3 "~" H 1850 1950 50  0001 C CNN
 	1    1850 1950
@@
 F 0 "R?" V 1750 1850 50  0000 C CNN
 F 1 "R" V 1850 1850 50  0000 C CNN
-F 2 "" V 1780 1850 50  0001 C CNN
+F 2 "Resistor_SMD:R_1206_3216Metric" V 1780 1850 50  0001 C CNN
 F 3 "~" H 1850 1850 50  0001 C CNN
 	1    1850 1850
@@
 F 0 "R?" V 2100 1700 50  0000 C CNN
 F 1 "R" V 2000 1700 50  0000 C CNN
-F 2 "" V 1930 1700 50  0001 C CNN
+F 2 "Resistor_SMD:R_1206_3216Metric" V 1930 1700 50  0001 C CNN
 F 3 "~" H 2000 1700 50  0001 C CNN
 	1    2000 1700
@@
 F 0 "C?" H 1965 7046 50  0000 L CNN
 F 1 "C" H 1965 6955 50  0000 L CNN
-F 2 "" H 1888 6850 50  0001 C CNN
+F 2 "Capacitor_SMD:C_1206_3216Metric" H 1888 6850 50  0001 C CNN
 F 3 "~" H 1850 7000 50  0001 C CNN
 	1    1850 7000
@@
 F 0 "C?" H 1615 7046 50  0000 L CNN
 F 1 "C" H 1615 6955 50  0000 L CNN
-F 2 "" H 1538 6850 50  0001 C CNN
+F 2 "Capacitor_SMD:C_1206_3216Metric" H 1538 6850 50  0001 C CNN
 F 3 "~" H 1500 7000 50  0001 C CNN
 	1    1500 7000
@@
 F 0 "C?" H 3215 7046 50  0000 L CNN
 F 1 "C" H 3215 6955 50  0000 L CNN
-F 2 "" H 3138 6850 50  0001 C CNN
+F 2 "Capacitor_SMD:C_1206_3216Metric" H 3138 6850 50  0001 C CNN
 F 3 "~" H 3100 7000 50  0001 C CNN
 	1    3100 7000
@@
 F 0 "C?" H 2865 7046 50  0000 L CNN
 F 1 "C" H 2865 6955 50  0000 L CNN
-F 2 "" H 2788 6850 50  0001 C CNN
+F 2 "Capacitor_SMD:C_1206_3216Metric" H 2788 6850 50  0001 C CNN
 F 3 "~" H 2750 7000 50  0001 C CNN
 	1    2750 7000
@@
 F 0 "R?" H 10220 1246 50  0000 L CNN
 F 1 "R" H 10220 1155 50  0000 L CNN
-F 2 "" V 10080 1200 50  0001 C CNN
+F 2 "Resistor_SMD:R_1206_3216Metric" V 10080 1200 50  0001 C CNN
 F 3 "~" H 10150 1200 50  0001 C CNN
 	1    10150 1200
@@
 F 0 "D?" V 8239 1633 50  0000 R CNN
 F 1 "LED" V 8148 1633 50  0000 R CNN
-F 2 "" H 8200 1750 50  0001 C CNN
+F 2 "LED_SMD:LED_1206_3216Metric" H 8200 1750 50  0001 C CNN
 F 3 "~" H 8200 1750 50  0001 C CNN
 	1    8200 1750
@@
 F 0 "R?" V 3400 2000 50  0000 C CNN
 F 1 "R" V 3500 2000 50  0000 C CNN
-F 2 "" V 3430 2000 50  0001 C CNN
+F 2 "Capacitor_SMD:C_1206_3216Metric" V 3430 2000 50  0001 C CNN
 F 3 "~" H 3500 2000 50  0001 C CNN
 	1    3500 2000
@@
 F 0 "C?" H 4915 6996 50  0000 L CNN
 F 1 "C" H 4915 6905 50  0000 L CNN
-F 2 "" H 4838 6800 50  0001 C CNN
+F 2 "Capacitor_SMD:C_1206_3216Metric" H 4838 6800 50  0001 C CNN
 F 3 "~" H 4800 6950 50  0001 C CNN
 	1    4800 6950
@@
 F 0 "C?" H 5265 6996 50  0000 L CNN
 F 1 "C" H 5265 6905 50  0000 L CNN
-F 2 "" H 5188 6800 50  0001 C CNN
+F 2 "Capacitor_SMD:C_1206_3216Metric" H 5188 6800 50  0001 C CNN
 F 3 "~" H 5150 6950 50  0001 C CNN
 	1    5150 6950
@@
 F 0 "C?" H 5665 6996 50  0000 L CNN
 F 1 "C" H 5665 6905 50  0000 L CNN
-F 2 "" H 5588 6800 50  0001 C CNN
+F 2 "Capacitor_SMD:C_1206_3216Metric" H 5588 6800 50  0001 C CNN
 F 3 "~" H 5550 6950 50  0001 C CNN
 	1    5550 6950
@@
 F 0 "C?" H 6015 6996 50  0000 L CNN
 F 1 "C" H 6015 6905 50  0000 L CNN
-F 2 "" H 5938 6800 50  0001 C CNN
+F 2 "Capacitor_SMD:C_1206_3216Metric" H 5938 6800 50  0001 C CNN
 F 3 "~" H 5900 6950 50  0001 C CNN
 	1    5900 6950
@@
 F 0 "R?" V 1993 3750 50  0000 C CNN
 F 1 "R" V 2084 3750 50  0000 C CNN
-F 2 "" V 2130 3750 50  0001 C CNN
+F 2 "Resistor_SMD:R_1206_3216Metric" V 2130 3750 50  0001 C CNN
 F 3 "~" H 2200 3750 50  0001 C CNN
 	1    2200 3750
@@
 F 0 "R?" V 1093 3750 50  0000 C CNN
 F 1 "R" V 1184 3750 50  0000 C CNN
-F 2 "" V 1230 3750 50  0001 C CNN
+F 2 "Resistor_SMD:R_1206_3216Metric" V 1230 3750 50  0001 C CNN
 F 3 "~" H 1300 3750 50  0001 C CNN
 	1    1300 3750
