File: Electronics/MidiControllerV1/MidiControllerV1.kicad_pcb (KiCad board)
At the start: 2 copper layers, 134 x 28 mm, 14 parts, among them J2 KeypadConnector, J3 OledConnector, J4 BluePillHeaderA, J5 BluepillHeaderB, SW1 Rotary_Encoder_Switch, SW2 Rotary_Encoder_Switch

Commit message: #32 Updated pcb v1
Connections:
- J3 pad 1: LCD_SCL -> LCD_SDA
- J3 pad 2: LCD_SDA -> LCD_SCL
- SW1 pad MP: GND -> (no net)
- SW2 pad MP: GND -> (no net)
Routing:
- net GND: track 9.21 -> 21.8 mm, vias 0 -> 67
- net +3V3: track 180.1 -> 182.1 mm
- net LCD_SDA: track 62.5 -> 63.9 mm, vias 0 -> 1
- added copper zone on B.Cu, net GND
